File: media-controller.sch (KiCad schematic (older format))
At the start: 4 parts, among them X1 XTAL_GND

Commit message: Add decoupling capacitors, usb port and reset switch
Parts:
- added C3, C4, C5, C6: 0.1u, symbol Device:C_Small
- added C7: 4.7u, symbol Device:C_Small
- added C8: 1u, symbol Device:C_Small
- added J1: USB_mini_micro_B, symbol tmk:USB_mini_micro_B
- added R1, R2: 10k, symbol tmk:R
- added R3, R4: 22, symbol tmk:R
- added SW1: SW_PUSH, symbol tmk:SW_PUSH
- gave numbers to parts that had none: 1
Connections:
- wire segments 14 -> 66

Commit message: Finish 2x2 media controller
Parts:
- added D1, D2, D3, D4: D, symbol Device:D
- added K1, K2, K3, K4: KEYSW, symbol tmk:KEYSW
Connections:
- net labels added: col0, col1, row0, row1
- wire segments 66 -> 87
- no-connect marks 0 -> 22
Changed lines of the file:
@@
 EESchema Schematic File Version 4
-EELAYER 29 0
+EELAYER 30 0
 EELAYER END
 $Descr A4 11693 8268
@@
 Wire Wire Line
 	7300 2950 6850 2950
+$Comp
+L tmk:KEYSW K1
+U 1 1 5F3AD3A5
+P 8750 1800
+F 0 "K1" H 8750 2033 60  0000 C CNN
+F 1 "KEYSW" H 8750 1700 60  0001 C CNN
+F 2 "" H 8750 1800 60  0000 C CNN
+F 3 "" H 8750 1800 60  0000 C CNN
+	1    8750 1800
+	1    0    0    -1
+$EndComp
+$Comp
+L tmk:KEYSW K3
+U 1 1 5F3ADED8
+P 9600 1800
+F 0 "K3" H 9600 2033 60  0000 C CNN
+F 1 "KEYSW" H 9600 1700 60  0001 C CNN
+F 2 "" H 9600 1800 60  0000 C CNN
+F 3 "" H 9600 1800 60  0000 C CNN
+	1    9600 1800
+	1    0    0    -1
+$EndComp
+$Comp
+L tmk:KEYSW K2
+U 1 1 5F3AE846
+P 8750 2550
+F 0 "K2" H 8750 2783 60  0000 C CNN
+F 1 "KEYSW" H 8750 2450 60  0001 C CNN
+F 2 "" H 8750 2550 60  0000 C CNN
+F 3 "" H 8750 2550 60  0000 C CNN
+	1    8750 2550
+	1    0    0    -1
+$EndComp
+$Comp
+L tmk:KEYSW K4
+U 1 1 5F3AF28D
+P 9600 2550
+F 0 "K4" H 9600 2783 60  0000 C CNN
+F 1 "KEYSW" H 9600 2450 60  0001 C CNN
+F 2 "" H 9600 2550 60  0000 C CNN
+F 3 "" H 9600 2550 60  0000 C CNN
+	1    9600 2550
+	1    0    0    -1
+$EndComp
+$Comp
+L Device:D D1
+U 1 1 5F3B2ADC
+P 8350 2050
+F 0 "D1" V 8396 1970 50  0000 R CNN
+F 1 "D" V 8305 1970 50  0000 R CNN
+F 2 "" H 8350 2050 50  0001 C CNN
+F 3 "~" H 8350 2050 50  0001 C CNN
+	1    8350 2050
+	0    -1   -1   0
+$EndComp
+$Comp
+L Device:D D3
+U 1 1 5F3B4F70
+P 9200 2050
+F 0 "D3" V 9246 1970 50  0000 R CNN
+F 1 "D" V 9155 1970 50  0000 R CNN
+F 2 "" H 9200 2050 50  0001 C CNN
+F 3 "~" H 9200 2050 50  0001 C CNN
+	1    9200 2050
+	0    -1   -1   0
+$EndComp
+$Comp
+L Device:D D2
+U 1 1 5F3B701A
+P 8350 2800
+F 0 "D2" V 8396 2720 50  0000 R CNN
+F 1 "D" V 8305 2720 50  0000 R CNN
+F 2 "" H 8350 2800 50  0001 C CNN
+F 3 "~" H 8350 2800 50  0001 C CNN
+	1    8350 2800
+	0    -1   -1   0
+$EndComp
+$Comp
+L Device:D D4
+U 1 1 5F3B794E
+P 9200 2800
+F 0 "D4" V 9246 2720 50  0000 R CNN
+F 1 "D" V 9155 2720 50  0000 R CNN
+F 2 "" H 9200 2800 50  0001 C CNN
+F 3 "~" H 9200 2800 50  0001 C CNN
+	1    9200 2800
+	0    -1   -1   0
+$EndComp
+Wire Wire Line
+	8450 1800 8350 1800
+Wire Wire Line
+	8350 1800 8350 1900
+Wire Wire Line
+	9050 1800 9050 2550
+Wire Wire Line
+	9900 1800 9900 2550
+Wire Wire Line
+	9300 1800 9200 1800
+Wire Wire Line
+	9200 1800 9200 1900
+Wire Wire Line
+	9200 2200 9200 2300
+Wire Wire Line
+	9200 2300 8350 2300
+Wire Wire Line
+	8350 2300 8350 2200
+Wire Wire Line
+	8350 2950 8350 3050
+Wire Wire Line
+	8350 3050 9200 3050
+Wire Wire Line
+	9200 3050 9200 2950
+Wire Wire Line
+	9200 2650 9200 2550
+Wire Wire Line
+	9200 2550 9300 2550
+Wire Wire Line
+	8350 2650 8350 2550
+Wire Wire Line
+	8350 2550 8450 2550
+Text Label 9050 1650 0    50   ~ 0
+col0
+Text Label 9900 1650 0    50   ~ 0
+col1
+Text Label 8150 2300 0    50   ~ 0
+row0
+Text Label 8150 3050 0    50   ~ 0
+row1
+Wire Wire Line
+	8350 2300 8150 2300
+Connection ~ 8350 2300
+Wire Wire Line
+	8350 3050 8150 3050
+Connection ~ 8350 3050
+Text Label 6850 2350 0    50   ~ 0
+row0
+Text Label 6850 2450 0    50   ~ 0
+row1
+Text Label 6850 2550 0    50   ~ 0
+col0
+Text Label 6850 2650 0    50   ~ 0
+col1
+NoConn ~ 6850 2250
+NoConn ~ 6850 2750
+NoConn ~ 6850 2850
+NoConn ~ 6850 3250
+NoConn ~ 6850 3350
+NoConn ~ 6850 3450
+NoConn ~ 6850 3550
+NoConn ~ 6850 3650
+NoConn ~ 6850 3750
+NoConn ~ 6850 3850
+NoConn ~ 6850 3950
+NoConn ~ 4700 3750
+NoConn ~ 4700 3850
+NoConn ~ 4700 3950
+NoConn ~ 4700 4050
+NoConn ~ 4700 4150
+NoConn ~ 4700 3150
+NoConn ~ 4700 3050
+NoConn ~ 4700 2950
+NoConn ~ 4700 2850
+NoConn ~ 4700 2750
+NoConn ~ 4700 2050
+$Comp
+L power:VCC #PWR?
+U 1 1 5F3FCCC3
+P 4150 2650
+F 0 "#PWR?" H 4150 2500 50  0001 C CNN
+F 1 "VCC" V 4165 2777 50  0000 L CNN
+F 2 "" H 4150 2650 50  0001 C CNN
+F 3 "" H 4150 2650 50  0001 C CNN
+	1    4150 2650
+	0    -1   -1   0
+$EndComp
+Wire Wire Line
+	4700 2650 4150 2650
+Wire Wire Line
+	9050 1800 9050 1650
+Connection ~ 9050 1800
+Wire Wire Line
+	9900 1650 9900 1800
+Connection ~ 9900 1800
 $EndSCHEMATC

Commit message: Use Device:Crystal_GND24 component
Parts:
- removed X1: XTAL_GND, symbol tmk:XTAL_GND
- added Y1: Crystal_GND24, symbol Device:Crystal_GND24
Connections:
- wire segments 87 -> 95
Changed lines of the file:
@@
 $EndComp
-$Comp
-L tmk:XTAL_GND X1
-U 1 1 5EBC62CF
-P 3600 3750
-F 0 "X1" H 3600 4042 60  0000 C CNN
-F 1 "XTAL_GND" H 3600 3936 60  0000 C CNN
-F 2 "" H 3600 3750 60  0000 C CNN
-F 3 "" H 3600 3750 60  0000 C CNN
-	1    3600 3750
-	1    0    0    -1
-$EndComp
-$Comp
-L Device:C_Small C1
-U 1 1 5EBC6863
-P 3200 3950
-F 0 "C1" H 3292 3996 50  0000 L CNN
-F 1 "22p" H 3292 3905 50  0000 L CNN
-F 2 "" H 3200 3950 50  0001 C CNN
-F 3 "~" H 3200 3950 50  0001 C CNN
-	1    3200 3950
-	1    0    0    -1
-$EndComp
-$Comp
-L Device:C_Small C2
-U 1 1 5EBC6EBF
-P 4000 3950
-F 0 "C2" H 4092 3996 50  0000 L CNN
-F 1 "22p" H 4092 3905 50  0000 L CNN
-F 2 "" H 4000 3950 50  0001 C CNN
-F 3 "~" H 4000 3950 50  0001 C CNN
-	1    4000 3950
-	1    0    0    -1
-$EndComp
-Wire Wire Line
-	4000 3850 4000 3750
-Wire Wire Line
-	4000 3750 3900 3750
-Wire Wire Line
-	3300 3750 3200 3750
-Wire Wire Line
-	3200 3750 3200 3850
-Wire Wire Line
-	3200 4050 3200 4150
-Wire Wire Line
-	4000 4150 4000 4050
-Wire Wire Line
-	3200 4150 3600 4150
-Wire Wire Line
-	3600 4150 3600 3950
-Connection ~ 3600 4150
-Wire Wire Line
-	3600 4150 4000 4150
-Wire Wire Line
-	4000 3750 4000 3650
-Connection ~ 4000 3750
-Wire Wire Line
-	4700 3550 3200 3550
-Wire Wire Line
-	3200 3550 3200 3750
-Connection ~ 3200 3750
-Wire Wire Line
-	4000 3650 4700 3650
 $Comp
 L power:VCC #PWR?
@@
 	1400 1750 1400 1850
 Connection ~ 1400 1750
-$Comp
-L power:GND #PWR?
-U 1 1 5EBE33A3
-P 3600 4350
-F 0 "#PWR?" H 3600 4100 50  0001 C CNN
-F 1 "GND" H 3605 4177 50  0000 C CNN
-F 2 "" H 3600 4350 50  0001 C CNN
-F 3 "" H 3600 4350 50  0001 C CNN
-	1    3600 4350
-	1    0    0    -1
-$EndComp
-Wire Wire Line
-	3600 4350 3600 4150
 Wire Wire Line
 	6850 3150 7000 3150
@@
 	9900 1650 9900 1800
 Connection ~ 9900 1800
+$Comp
+L Device:Crystal_GND24 Y1
+U 1 1 5F412834
+P 2650 4300
+F 0 "Y1" H 2844 4346 50  0000 L CNN
+F 1 "Crystal_GND24" H 2844 4255 50  0000 L CNN
+F 2 "" H 2650 4300 50  0001 C CNN
+F 3 "~" H 2650 4300 50  0001 C CNN
+	1    2650 4300
+	1    0    0    -1
+$EndComp
+$Comp
+L Device:C_Small C1
+U 1 1 5F4169CC
+P 2200 4300
+F 0 "C1" V 1971 4300 50  0000 C CNN
+F 1 "22p" V 2062 4300 50  0000 C CNN
+F 2 "" H 2200 4300 50  0001 C CNN
+F 3 "~" H 2200 4300 50  0001 C CNN
+	1    2200 4300
+	0    1    1    0
+$EndComp
+$Comp
+L power:GND #PWR?
+U 1 1 5F4190B2
+P 2650 3850
+F 0 "#PWR?" H 2650 3600 50  0001 C CNN
+F 1 "GND" H 2655 3677 50  0000 C CNN
+F 2 "" H 2650 3850 50  0001 C CNN
+F 3 "" H 2650 3850 50  0001 C CNN
+	1    2650 3850
+	-1   0    0    1
+$EndComp
+Wire Wire Line
+	2650 4100 2650 3950
+$Comp
+L power:GND #PWR?
+U 1 1 5F41B6D8
+P 2650 4750
+F 0 "#PWR?" H 2650 4500 50  0001 C CNN
+F 1 "GND" H 2655 4577 50  0000 C CNN
+F 2 "" H 2650 4750 50  0001 C CNN
+F 3 "" H 2650 4750 50  0001 C CNN
+	1    2650 4750
+	1    0    0    -1
+$EndComp
+Wire Wire Line
+	2650 4500 2650 4600
+Wire Wire Line
+	2100 4300 2000 4300
+Wire Wire Line
+	2000 4300 2000 4600
+Wire Wire Line
+	2000 4600 2650 4600
+Connection ~ 2650 4600
+Wire Wire Line
+	2650 4600 2650 4750
+Wire Wire Line
+	2000 4300 2000 3950
+Wire Wire Line
+	2000 3950 2650 3950
+Connection ~ 2000 4300
+Connection ~ 2650 3950
+Wire Wire Line
+	2650 3950 2650 3850
+$Comp
+L Device:C_Small C2
+U 1 1 5F42281A
+P 3100 4300
+F 0 "C2" V 2871 4300 50  0000 C CNN
+F 1 "22p" V 2962 4300 50  0000 C CNN
+F 2 "" H 3100 4300 50  0001 C CNN
+F 3 "~" H 3100 4300 50  0001 C CNN
+	1    3100 4300
+	0    1    1    0
+$EndComp
+Wire Wire Line
+	2800 4300 2900 4300
+Wire Wire Line
+	2650 4600 3300 4600
+Wire Wire Line
+	3300 4600 3300 4300
+Wire Wire Line
+	3300 4300 3200 4300
+Wire Wire Line
+	3300 4300 3300 3950
+Wire Wire Line
+	3300 3950 2650 3950
+Connection ~ 3300 4300
+Wire Wire Line
+	2300 4300 2400 4300
+Wire Wire Line
+	2400 4300 2400 3550
+Wire Wire Line
+	2400 3550 4700 3550
+Connection ~ 2400 4300
+Wire Wire Line
+	2400 4300 2500 4300
+Wire Wire Line
+	2900 4300 2900 3650
+Wire Wire Line
+	2900 3650 4700 3650
+Connection ~ 2900 4300
+Wire Wire Line
+	2900 4300 3000 4300
 $EndSCHEMATC

Commit message: Add rotary encoder
Parts:
- added SW2: Rotary_Encoder, symbol Device:Rotary_Encoder
Connections:
- net labels added: EN1, EN2
- wire segments 95 -> 96
- no-connect marks 22 -> 20
Changed lines of the file:
@@
 NoConn ~ 4700 4150
 NoConn ~ 4700 3150
-NoConn ~ 4700 3050
-NoConn ~ 4700 2950
 NoConn ~ 4700 2850
 NoConn ~ 4700 2750
@@
 Wire Wire Line
 	2900 4300 3000 4300
+$Comp
+L Device:Rotary_Encoder SW2
+U 1 1 5F43CD25
+P 8850 4000
+F 0 "SW2" H 9080 4046 50  0000 L CNN
+F 1 "Rotary_Encoder" H 9080 3955 50  0000 L CNN
+F 2 "" H 8700 4160 50  0001 C CNN
+F 3 "~" H 8850 4260 50  0001 C CNN
+	1    8850 4000
+	1    0    0    -1
+$EndComp
+$Comp
+L power:GND #PWR?
+U 1 1 5F43D951
+P 8350 4000
+F 0 "#PWR?" H 8350 3750 50  0001 C CNN
+F 1 "GND" V 8355 3872 50  0000 R CNN
+F 2 "" H 8350 4000 50  0001 C CNN
+F 3 "" H 8350 4000 50  0001 C CNN
+	1    8350 4000
+	0    1    1    0
+$EndComp
+Wire Wire Line
+	8350 4000 8550 4000
+Text Label 8550 4100 2    50   ~ 0
+EN1
+Text Label 8550 3900 2    50   ~ 0
+EN2
+Text Label 4700 3050 2    50   ~ 0
+EN1
+Text Label 4700 2950 2    50   ~ 0
+EN2
 $EndSCHEMATC
